Commit message: feat : show robot.urdf on rviz2

File: ekf_tf_bringup/urdf/robot.urdf (robot description, URDF)
Before this commit: robot mecanum_robot, 7 links, 6 joints
Links:
- added link laser
Joints:
- added joint merged_laser_joint: type fixed, parent base_link, child laser, origin xyz=0 0 0.66 rpy=0 0 0
